Commit message: Add ZED X Nano description
Co-authored-by: Copilot <copilot@github.com>

File: urdf/include/materials.urdf.xacro (robot description, xacro)
@@ -34,4 +34,7 @@
         <color rgba="0.25 0.25 0.25 1.0"/>
     </material>
+    <material name="zedxnano_mat">
+        <color rgba="0.25 0.25 0.25 1.0"/>
+    </material>
     <material name="zedxhdr_mat">
         <color rgba="0.25 0.25 0.25 1.0"/>

File: urdf/zed_macro.urdf.xacro (robot description, xacro)
@@ -85,4 +85,13 @@
       <xacro:property name="screw_offset_x" value="0.0" />
       <xacro:property name="screw_offset_z" value="-0.016" />
+      <xacro:property name="optical_offset_x" value="-0.01" />
+      <xacro:property name="mono" value="false" />
+    </xacro:if>
+    <xacro:if value="${model == 'zedxnano'}">
+      <xacro:property name="baseline" value="0.018" />
+      <xacro:property name="height" value="0.0305" />
+      <xacro:property name="bottom_slope" value="0.0" />
+      <xacro:property name="screw_offset_x" value="0.0" />
+      <xacro:property name="screw_offset_z" value="-0.01525" />
       <xacro:property name="optical_offset_x" value="-0.01" />
       <xacro:property name="mono" value="false" />
