Commit message: Add ZED X One S model and description

File: urdf/include/materials.urdf.xacro (robot description, xacro)
@@ -52,4 +52,7 @@
         <color rgba="0.25 0.25 0.25 1.0"/>
     </material>
+    <material name="zedxones_mat">
+        <color rgba="0.25 0.25 0.25 1.0"/>
+    </material>
     <material name="zedxone4k_mat">
         <color rgba="0.25 0.25 0.25 1.0"/>

File: urdf/zed_macro.urdf.xacro (robot description, xacro)
@@ -130,4 +130,13 @@
       <xacro:property name="screw_offset_x" value="0.0" />
       <xacro:property name="screw_offset_z" value="-0.0155" />
+      <xacro:property name="optical_offset_x" value="-0.005" />
+      <xacro:property name="mono" value="true" />
+    </xacro:if>
+    <xacro:if value="${model == 'zedxones'}">
+      <xacro:property name="baseline" value="0.0" />
+      <xacro:property name="height" value="0.025" />
+      <xacro:property name="bottom_slope" value="0.0" />
+      <xacro:property name="screw_offset_x" value="0.0" />
+      <xacro:property name="screw_offset_z" value="-0.0125" />
       <xacro:property name="optical_offset_x" value="0.0" />
       <xacro:property name="mono" value="true" />
