Commit message: Add zexconecore

File: urdf/zed_macro.urdf.xacro (robot description, xacro)
@@ -171,4 +171,14 @@
       <xacro:property name="screw_offset_z" value="-0.0125" />
       <xacro:property name="optical_offset_x" value="0.0" />
+      <xacro:property name="mono" value="true" />
+      <xacro:property name="mat" value="0.25 0.25 0.25 1.0" />
+    </xacro:if>
+    <xacro:if value="${model == 'zedxonecore'}">
+      <xacro:property name="baseline" value="0.0" />
+      <xacro:property name="height" value="0.027" />
+      <xacro:property name="bottom_slope" value="0.0" />
+      <xacro:property name="screw_offset_x" value="0.00" />
+      <xacro:property name="screw_offset_z" value="-0.0135" />
+      <xacro:property name="optical_offset_x" value="0.00086" />
       <xacro:property name="mono" value="true" />
       <xacro:property name="mat" value="0.25 0.25 0.25 1.0" />

Commit message: Fix optical frame offset values

File: urdf/zed_macro.urdf.xacro (robot description, xacro)
@@ -30,5 +30,5 @@
       <xacro:property name="screw_offset_x" value="0.0" />
       <xacro:property name="screw_offset_z" value="0.0" />
-      <xacro:property name="optical_offset_x" value="-0.01" />
+      <xacro:property name="optical_offset_x" value="-0.005" />
       <xacro:property name="mono" value="false" />
       <xacro:property name="mat" value="0.8 0.8 0.8 1.0" />
@@ -50,5 +50,5 @@
       <xacro:property name="screw_offset_x" value="0.0" />
       <xacro:property name="screw_offset_z" value="0.0" />
-      <xacro:property name="optical_offset_x" value="-0.01" />
+      <xacro:property name="optical_offset_x" value="-0.005" />
       <xacro:property name="mono" value="false" />
       <xacro:property name="mat" value="0.25 0.25 0.25 1.0" />
@@ -60,5 +60,5 @@
       <xacro:property name="screw_offset_x" value="-0.01" />
       <xacro:property name="screw_offset_z" value="0.0" />
-      <xacro:property name="optical_offset_x" value="-0.01" />
+      <xacro:property name="optical_offset_x" value="-0.005" />
       <xacro:property name="mono" value="false" />
       <xacro:property name="mat" value="0.25 0.25 0.25 1.0" />
@@ -70,5 +70,5 @@
       <xacro:property name="screw_offset_x" value="0.0" />
       <xacro:property name="screw_offset_z" value="-0.016" />
-      <xacro:property name="optical_offset_x" value="-0.01" />
+      <xacro:property name="optical_offset_x" value="-0.005" />
       <xacro:property name="mono" value="false" />
       <xacro:property name="mat" value="0.25 0.25 0.25 1.0" />
@@ -80,5 +80,5 @@
       <xacro:property name="screw_offset_x" value="0.0" />
       <xacro:property name="screw_offset_z" value="-0.016" />
-      <xacro:property name="optical_offset_x" value="-0.01" />
+      <xacro:property name="optical_offset_x" value="-0.005" />
       <xacro:property name="mono" value="false" />
       <xacro:property name="mat" value="0.25 0.25 0.25 1.0" />
@@ -90,5 +90,5 @@
       <xacro:property name="screw_offset_x" value="0.0" />
       <xacro:property name="screw_offset_z" value="-0.016" />
-      <xacro:property name="optical_offset_x" value="-0.01" />
+      <xacro:property name="optical_offset_x" value="-0.005" />
       <xacro:property name="mono" value="false" />
       <xacro:property name="mat" value="0.25 0.25 0.25 1.0" />
@@ -100,5 +100,5 @@
       <xacro:property name="screw_offset_x" value="0.0" />
       <xacro:property name="screw_offset_z" value="-0.01525" />
-      <xacro:property name="optical_offset_x" value="-0.01" />
+      <xacro:property name="optical_offset_x" value="-0.0035" />
       <xacro:property name="mono" value="false" />
       <xacro:property name="mat" value="0.25 0.25 0.25 1.0" />
@@ -110,5 +110,5 @@
       <xacro:property name="screw_offset_x" value="0.0" />
       <xacro:property name="screw_offset_z" value="-0.016" />
-      <xacro:property name="optical_offset_x" value="-0.01" />
+      <xacro:property name="optical_offset_x" value="-0.005" />
       <xacro:property name="mono" value="false" />
       <xacro:property name="mat" value="0.25 0.25 0.25 1.0" />
@@ -120,5 +120,5 @@
       <xacro:property name="screw_offset_x" value="0.0" />
       <xacro:property name="screw_offset_z" value="-0.016" />
-      <xacro:property name="optical_offset_x" value="-0.01" />
+      <xacro:property name="optical_offset_x" value="-0.005" />
       <xacro:property name="mono" value="false" />
       <xacro:property name="mat" value="0.25 0.25 0.25 1.0" />
